Commit message: V2

File: 1dHopper_withoutBeam2.urdf (robot description, URDF)
Before this commit: robot 1dhopper, 6 links, 5 joints
Links:
- link balance_beam: mass 6 -> 2; geometry collision cylinder length=1 radius=0.02; visual cylinder length=1 radius=0.02
- link base_link: mass 0.15 -> 0.2
- link left_weight: mass 1.5 -> 1
- link leg: mass 0.15 -> 0.45
- link right_weight: mass 1.5 -> 1
Joints:
- joint base_to_beam: child base_link -> balance_beam; parent balance_beam -> base_link; type revolute -> continuous

File: backwardVersion/1dHopper_withoutBeam.urdf (robot description, URDF)
Before this commit: robot 1dhopper, 6 links, 5 joints
Links:
- link balance_beam: mass 6 -> 0.05; geometry collision cylinder length=1.5 radius=0.01; visual cylinder length=1.5 radius=0.01
- link left_weight: mass 1.5 -> 4
- link leg: mass 0.15 -> 0.45
- link right_weight: mass 1.5 -> 4
Joints:
- joint leftWeight_beam: origin xyz=0.5 0 -0.02 -> xyz=0.75 0 -0.02
- joint rightWeight_beam: origin xyz=-0.5 0 -0.02 -> xyz=-0.75 0 -0.02

File: v2/1dHopper_withoutBeam.urdf (robot description, URDF)
Before this commit: robot 1dhopper, 6 links, 5 joints
Links:
- link balance_beam: mass 6 -> 5
