Commit message: Position+Torque control

File: 1dHopper_withoutBeam.urdf (robot description, URDF)
Before this commit: robot 1dhopper, 6 links, 5 joints
Joints:
- joint base_to_beam: limit lower=-1.57079632679 upper=1.57079632679 effort=1000.0 velocity=100 -> lower=-0.471 upper=0.471 effort=1000.0 velocity=100
