Commit message: Real time control suite

File: 3D version/1dHopper_withoutBeam.urdf (robot description, URDF)
Before this commit: robot 1dhopper, 5 links, 4 joints
Links:
- removed link upper_base_link
- added link left_weight, mass 1.5; collision cylinder length=0.1 radius=0.04; visual cylinder length=0.1 radius=0.04
- added link right_weight, mass 1.5; collision cylinder length=0.1 radius=0.04; visual cylinder length=0.1 radius=0.04
- link balance_beam: geometry collision cylinder length=1 radius=0.01; visual cylinder length=1 radius=0.01
Joints:
- removed joint base_joint
- added joint leftWeight_beam: type fixed, parent balance_beam, child left_weight, origin xyz=0.5 0 -0.02
- added joint rightWeight_beam: type fixed, parent balance_beam, child right_weight, origin xyz=-0.5 0 -0.02
- joint base_to_beam: child upper_base_link -> base_link; origin xyz=0 0 -0.1 -> xyz=0 0 0
