Commit message: FPS View

File: 3D version/3dHopper.urdf (robot description, URDF)
Before this commit: robot 1dhopper, 5 links, 4 joints
Links:
- link balance_beam: mass 6 -> 16

Commit message: Stable hopping height

File: 3D version/3dHopper.urdf (robot description, URDF)
Before this commit: robot 1dhopper, 5 links, 4 joints
Joints:
- joint base_joint: limit lower=-0.471 upper=0.471 effort=1000.0 velocity=100 -> lower=-0.349 upper=0.349 effort=1000.0 velocity=100
- joint base_to_beam: limit lower=-0.471 upper=0.471 effort=1000.0 velocity=100 -> lower=-0.523 upper=0.523 effort=1000.0 velocity=100; origin xyz=0 0 -0.1 -> xyz=0 0 -0.25

Commit message: BodyAttitudeControl

File: 3D version/3dHopper.urdf (robot description, URDF)
Before this commit: robot 1dhopper, 5 links, 4 joints
Joints:
- joint base_joint: type revolute -> continuous
- joint base_to_beam: type revolute -> continuous

Commit message: REcail

File: 3D version/3dHopper.urdf (robot description, URDF)
Before this commit: robot 1dhopper, 5 links, 4 joints
Links:
- link leg: mass 0.15 -> 0.91
Joints:
- joint base_joint: type continuous -> revolute
- joint base_to_beam: limit lower=-0.523 upper=0.523 effort=1000.0 velocity=100 -> lower=-0.349 upper=0.349 effort=1000.0 velocity=100; type continuous -> revolute
